File: daemon_v0.kicad_pcb (KiCad board)
At the start: 4 copper layers, 85.6 x 54 mm, 282 parts, among them J1 PTC_2A, J10 USB_A, J11 USB_C_Receptacle, J12 WAGO-2060-404, J13 Goobay-74446, J14 HR911105A, J15 SJ2-2531X, J16 Speaker, J17 Analog-In, J18 RS485-Bus, J19 UART-Debug, J2 10m, J3 Radxa-40Pin, J4 AUX-GPIO, J6 ST7789V2, J7 USB_C_Plug_USB2.0, J8 USB_A, J9 USB_A, Q1 BC857, Q2 BSS84, Q3 2N7002, Q4 AO3400A, SW1 SW_PWR, SW2 SKRHABE010, U1 IP5328P, U10 MAX98357A, U11 ISO1212, U12 USBLC6-2SC6, U13 INMP441, U14 SL2.1A, U15 SY6280AAC, U16 USBLC6-2SC6, U17 USBLC6-2SC6, U18 USBLC6-2SC6, U19 USBLC6-2SC6, U2 AP2112K-3.3, U20 USBLC6-2SC6, U21 PCF8574, U22 SY6280AAC, U23 74AHCT1G125, U24 INMP441, U25 ESD9B5.0ST5G, U26 ESD9B5.0ST5G, U27 NAU88C22, U28 ADS1115, U29 SP3485, U3 SL2.1A, U30 TSOP38238, U4 SY6280AAAC, U5 SY6280AAC, U6 SY6280AAC, U7 NE555DR, U8 CC1101, U9 RTL8152B, Y1 12MHz, Y2 12MHz, Y3 27MHz, Y4 25MHz

Commit message: fix: screen connector through-hole, female headers, antenna keepout
- J6 screen connector: PinSocket→PinHeader (through-hole, screen sits
  flush against PCB bottom)
- J17 (Analog-In), J18 (RS485), J19 (UART): male→female pin sockets
- Added antenna keep-out zone (16×16mm rectangle on Dwgs.User)
- Preserved 265 component placements from screenshot2
- All 4581 drawings preserved (Radxa DXF + custom shapes)

Co-Authored-By: Claude Opus 4.6 (1M context) <noreply@anthropic.com>
Parts:
- ANT1: value 0915AT43A0026 -> 915MHz Chip Antenna
- BAT1: value Li-ion -> Li-ion Battery
- D1: value SMBJ5.0A -> TVS 5V_SYS Clamp
- D10: value ESD5Z3.3 -> ESD Goobay CC1
- D11: value ESD5Z3.3 -> ESD Goobay CC2
- D2: value SMBJ5.0A -> TVS VIN Clamp
- D3: value ESD5Z3.3 -> ESD Port1 CC
- D4: value ESD5Z3.3 -> ESD Port5 CC1
- D5: value ESD5Z3.3 -> ESD Port5 CC2
- D6: value SS34 -> SS34 Charge Port1→VIN
- D7: value SS34 -> SS34 Charge Port4→VIN
- D8: value SS34 -> SS34 Charge Port5→VIN
- D9: value VCAN26A2 -> TVS ISO Input Clamp
- F1: value 60R -> PTC ISO Ch1 60Ω
- F2: value 60R -> PTC ISO Ch2 60Ω
- FB1: value BLM31PG601SN1L -> 5V_AUDIO Ferrite 1.5A
- FB2: value BLM18AG601SN1 -> MIC_VDD Ferrite
- J1: value PTC_2A -> Battery PTC 2A Fuse
- J10: value USB_A -> USB-A♂ Charge Port 4
- J11: value USB_C_Receptacle -> USB-C♀ Main Port 5
- J12: value WAGO-2060-404 -> WAGO 4P Field Terminal
- J13: value Goobay-74446 -> USB-C♀ Goobay Bridge
- J14: value HR911105A -> RJ45 MagJack
- J15: value SJ2-2531X -> TRRS 3.5mm Jack
- J16: value Speaker -> Speaker JST
- J17, J19: footprint PinHeader_1x04_P2.54mm_Vertical -> PinSocket_1x04_P2.54mm_Vertical
- J18: footprint PinHeader_1x03_P2.54mm_Vertical -> PinSocket_1x03_P2.54mm_Vertical
- J2: value 10m -> 10mΩ Current Sense
- J3: value Radxa-40Pin -> 40-Pin Radxa Header
- J4: value AUX-GPIO -> AUX GPIO Breakout
- J6: value ST7789V2 -> ST7789 SPI Display; footprint PinSocket_1x08_P2.54mm_Vertical -> PinHeader_1x08_P2.54mm_Vertical
- J7: value USB_C_Plug_USB2.0 -> USB-C♂ Plug → Radxa (KEY)
- J8: value USB_A -> USB-A♀ Host Port 2
- J9: value USB_A -> USB-A♀ Host Port 3
- L1: value 2u2 -> 2.2uH Boost Inductor
- LED1: value WS2812B-2020 -> WS2812B Status 1
- LED2: value WS2812B-2020 -> WS2812B Status 2
- LED3: value WS2812B-2020 -> WS2812B Status 3
- LED4: value WS2812B-2020 -> WS2812B Status 4
- LED5: value VSMB294008 -> IR Blaster LED
- LED6: value RED_0402 -> Mic Recording Red 1
- LED7: value RED_0402 -> Mic Recording Red 2
- LED8: value GREEN_0402 -> Power Green LED
- Q1: value BC857 -> BC857 Dummy Load PNP
- Q2: value BSS84 -> BSS84 Wake PMOS
- Q3: value 2N7002 -> 2N7002 PMIC Kill NMOS
- Q4: value AO3400A -> AO3400A IR Drive NMOS
- SW1: value SW_PWR -> Power Button
- SW2: value SKRHABE010 -> 5-Way Nav Switch
- TP1: value TP_VIN -> TP VIN
- TP2: value TP_BAT -> TP BAT
- TP3: value TP_LX -> TP LX
- TP4: value TP_VSYS -> TP VSYS
- U1: value IP5328P -> IP5328P PMIC
- U10: value MAX98357A -> MAX98357A I2S Amp
- U11: value ISO1212 -> ISO1212 Dual Isolator
- U12: value USBLC6-2SC6 -> ESD USB Port1
- U13: value INMP441 -> INMP441 Mic Left
- U14: value SL2.1A -> SL2.1A USB Hub 2
- U15: value SY6280AAC -> SY6280 Port4 USB-A♂
- U16: value USBLC6-2SC6 -> ESD USB Port2
- U17: value USBLC6-2SC6 -> ESD USB Port3
- U18: value USBLC6-2SC6 -> ESD USB Port4
- U19: value USBLC6-2SC6 -> ESD USB Port5
- U2: value AP2112K-3.3 -> AP2112K 3.3V LDO
- U20: value USBLC6-2SC6 -> ESD Goobay Bridge
- U21: value PCF8574 -> PCF8574 I2C GPIO Exp
- U22: value SY6280AAC -> SY6280 Port5 USB-C♀
- U23: value 74AHCT1G125 -> 3.3→5V Level Shifter
- U24: value INMP441 -> INMP441 Mic Right
- U3: value SL2.1A -> SL2.1A USB Hub 1
- U4: value SY6280AAAC -> SY6280 Port1 Radxa Key
- U5: value SY6280AAC -> SY6280 Port2 USB-A♀
- U6: value SY6280AAC -> SY6280 Port3 USB-A♀
- U7: value NE555DR -> NE555 Heartbeat Timer
- U8: value CC1101 -> CC1101 Sub-GHz Radio
- U9: value RTL8152B -> RTL8152B Ethernet
- Y1: value 12MHz -> 12MHz Hub1 Xtal
- Y2: value 12MHz -> 12MHz Hub2 Xtal
- Y3: value 27MHz -> 27MHz CC1101 Xtal
- Y4: value 25MHz -> 25MHz Ethernet Xtal
- moved LED5 292.0 mm to (65.5, 151.5), turned to 90 degrees
- moved LED4 274.4 mm to (129.1, 116.8), turned to -90 degrees
- moved C13 272.6 mm to (100.2, 166.0), turned to 180 degrees
- moved LED1 262.5 mm to (134.6, 111.2)
- moved LED3 261.5 mm to (134.6, 122.3)
- moved LED2 259.5 mm to (140.2, 116.8), turned to 90 degrees
- moved SW1 254.0 mm to (85.5, 101.7)
- moved SW2 253.3 mm to (134.6, 116.8)
- moved Y4 238.4 mm to (128.1, 130.7), turned to 180 degrees
- moved D1 236.7 mm to (59.6, 184.0)
- moved D10 236.7 mm to (71.7, 220.0)
- moved D11 236.7 mm to (83.7, 220.0)
- moved D2 236.7 mm to (71.7, 184.0)
- moved D3 236.7 mm to (47.6, 196.0)
- moved D4 236.7 mm to (59.6, 196.0)
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Other:
- board size 85.6 x 54 mm -> 91.5 x 53 mm
- board text added: "4"
- board text added: "ZER0 3W_V1.11"
- board text removed: "40"
- board text removed: "40-PIN GPIO HEADER"
- board text removed: "Inductor↔XTALs ≥15mm | Antenna keepout 5mm | MagJack↔USB-C ≥15mm"
- board text removed: "M2.5"
- board text removed: "RADXA ZERO 3W (underneath)"
- board text removed: "RULES: Power↔RF ≥20mm | Inductor↔RF ≥25mm | XTAL_26↔XTAL_25 ≥10mm"
- board text removed: "SD"
- board text removed: "SECONDARY COMPONENTS (111 passives) — don't touch, they follow their parent IC"
- board text removed: "USB-C HOST"
- board text removed: "USB-C OTG/PWR"
- board text removed: "WiFi U.FL"
- board text removed: "µHDMI"
- board text removed: "← 85.6 mm →"
- board text removed: "⚠ NO TALL PARTS ON B.Cu IN THIS ZONE"

Commit message: chore: KiCad re-import — 336 components, placements preserved
Re-imported netlist into KiCad PCB:
- 336/336 footprints placed (ATECC608B footprint fixed)
- 1096 pad-net connections
- 261 components in your placed positions (from screenshot2)
- 75 new protection/security components in staging area
- 4582 drawings preserved (Radxa DXF + custom shapes)

Co-Authored-By: Claude Opus 4.6 (1M context) <noreply@anthropic.com>
Parts:
- removed J18: RS485-Bus, PinSocket_1x03_P2.54mm_Vertical
- removed J19: UART-Debug, PinSocket_1x04_P2.54mm_Vertical
- added C119: 100n, C_0402_1005Metric, F.Cu at (240.0, 580.0)
- added C120: 100n, C_0402_1005Metric, F.Cu at (224.0, 588.0)
- added C121: 100n, C_0402_1005Metric, F.Cu at (232.0, 588.0)
- added C122: 100n, C_0402_1005Metric, F.Cu at (240.0, 588.0)
- added C123: 100n, C_0402_1005Metric, F.Cu at (248.0, 588.0)
- added C124: 100n, C_0402_1005Metric, F.Cu at (256.0, 588.0)
- added C125: 100n, C_0402_1005Metric, F.Cu at (264.0, 588.0)
- added D12: ESD5Z3.3, D_SOD-523, F.Cu at (212.0, 378.0)
- added D13: SMBJ5.0A, D_SMB, F.Cu at (224.0, 402.0)
- added D14: SMBJ5.0A, D_SMB, F.Cu at (236.0, 402.0)
- added D15: SMBJ5.0A, D_SMB, F.Cu at (248.0, 402.0)
- added D16: SS34, D_SMA, F.Cu at (200.0, 414.0)
- added D17: SMBJ5.0A, D_SMB, F.Cu at (212.0, 414.0)
- added D18: ESD5Z3.3, D_SOD-523, F.Cu at (224.0, 414.0)
- added D19: ESD5Z3.3, D_SOD-523, F.Cu at (236.0, 414.0)
- added D20: ESD5Z3.3, D_SOD-523, F.Cu at (248.0, 414.0)
- added D21: ESD5Z3.3, D_SOD-523, F.Cu at (260.0, 414.0)
- added D22: ESD5Z3.3, D_SOD-523, F.Cu at (272.0, 414.0)
- added D23: ESD5Z3.3, D_SOD-523, F.Cu at (284.0, 414.0)
- added D24: ESD5Z3.3, D_SOD-523, F.Cu at (200.0, 426.0)
- added D25: ESD5Z3.3, D_SOD-523, F.Cu at (212.0, 426.0)
- added D26: SM712, SOT-23-6, F.Cu at (224.0, 426.0)
- added D27: ESD5Z3.3, D_SOD-523, F.Cu at (260.0, 426.0)
- added D28: SM712, SOT-23-6, F.Cu at (272.0, 426.0)
- added D29: SM712, SOT-23-6, F.Cu at (284.0, 426.0)
- added D30: ESD5Z3.3, D_SOD-523, F.Cu at (200.0, 438.0)
- added D31: ESD5Z3.3, D_SOD-523, F.Cu at (212.0, 438.0)
- added D32: ESD5Z3.3, D_SOD-523, F.Cu at (224.0, 438.0)
- added D33: ESD5Z3.3, D_SOD-523, F.Cu at (236.0, 438.0)
- added D34: ESD5Z3.3, D_SOD-523, F.Cu at (248.0, 438.0)
- added D35: ESD5Z3.3, D_SOD-523, F.Cu at (260.0, 438.0)
- added F10: PTC_500mA, Fuse_0805_2012Metric, F.Cu at (284.0, 438.0)
- added F3: PTC_1A, Fuse_1206_3216Metric, F.Cu at (212.0, 402.0)
- added F4: PTC_500mA, Fuse_0805_2012Metric, F.Cu at (260.0, 402.0)
- added F5: PTC_500mA, Fuse_0805_2012Metric, F.Cu at (272.0, 402.0)
- added F6: PTC_500mA, Fuse_0805_2012Metric, F.Cu at (284.0, 402.0)
- added F7: PTC_200mA, Fuse_0805_2012Metric, F.Cu at (236.0, 426.0)
- added F8: PTC_200mA, Fuse_0805_2012Metric, F.Cu at (248.0, 426.0)
- added F9: PTC_500mA, Fuse_0805_2012Metric, F.Cu at (272.0, 438.0)
- added K1: G6K-2F-Y, Relay_DPDT_Omron_G6K-2F-Y, F.Cu at (240.0, 524.0)
- added Q5: AO3400A, SOT-23, F.Cu at (212.0, 390.0)
- added R66: 100, R_0402_1005Metric, F.Cu at (216.0, 580.0)
- added R67: 10k, R_0402_1005Metric, F.Cu at (248.0, 580.0)
- added R68: 10k, R_0402_1005Metric, F.Cu at (256.0, 580.0)
- added R69: 10k, R_0402_1005Metric, F.Cu at (264.0, 580.0)
- added R70: 10k, R_0402_1005Metric, F.Cu at (272.0, 580.0)
- added R71: 1k, R_0402_1005Metric, F.Cu at (280.0, 580.0)
- added R72: 1k, R_0402_1005Metric, F.Cu at (288.0, 580.0)
- added R73: 1k, R_0402_1005Metric, F.Cu at (200.0, 588.0)
- added R74: 1k, R_0402_1005Metric, F.Cu at (208.0, 588.0)
- added R75: 1k, R_0402_1005Metric, F.Cu at (216.0, 588.0)
- added U31: ATECC608B, DFN-8-1EP_2x3mm_P0.5mm_EP0.61x2.2mm, F.Cu at (260.0, 280.0)
- added U32: 74LVC04A, TSSOP-14_4.4x5mm_P0.65mm, F.Cu at (280.0, 280.0)
- added U33: TS3USB221, VSSOP-10_3x3mm_P0.5mm, F.Cu at (200.0, 300.0)
- added U34: TS3USB221, VSSOP-10_3x3mm_P0.5mm, F.Cu at (220.0, 300.0)
- added U35: TS3USB221, VSSOP-10_3x3mm_P0.5mm, F.Cu at (240.0, 300.0)
- added U36: TS3USB221, VSSOP-10_3x3mm_P0.5mm, F.Cu at (260.0, 300.0)
- added U37: TS3USB221, VSSOP-10_3x3mm_P0.5mm, F.Cu at (280.0, 300.0)
- D10: footprint D_SOD-523 -> SOT-323_SC-70
- D9: footprint SOT-323_SC-70 -> D_SOD-123
- J17: footprint PinSocket_1x04_P2.54mm_Vertical -> PinSocket_1x05_P2.54mm_Vertical
- J4: footprint PinSocket_2x04_P2.54mm_Vertical -> PinSocket_2x05_P2.54mm_Vertical
- R34, R36: footprint R_2512_6332Metric -> R_0402_1005Metric
- R35, R37: footprint R_0402_1005Metric -> R_2512_6332Metric
- R47: footprint R_1206_3216Metric -> R_0402_1005Metric
- R48: footprint R_0402_1005Metric -> R_1206_3216Metric
- R51: footprint R_0805_2012Metric -> R_0402_1005Metric
- R53: footprint R_0402_1005Metric -> R_0805_2012Metric
- moved R44 116.3 mm to (200.0, 548.0)
- moved C103 110.3 mm to (208.0, 564.0)
- moved C112 110.3 mm to (208.0, 572.0)
- moved C116 110.3 mm to (208.0, 580.0)
- moved C71 110.3 mm to (208.0, 532.0)
- moved C82 110.3 mm to (208.0, 540.0)
- moved C96 110.3 mm to (208.0, 556.0)
- moved C11 68.0 mm to (288.0, 460.0)
- moved C14 68.0 mm to (288.0, 468.0)
- moved C24 68.0 mm to (288.0, 476.0)
- moved C32 68.0 mm to (288.0, 484.0)
- moved C40 68.0 mm to (288.0, 492.0)
- moved C46 68.0 mm to (288.0, 500.0)
- moved C53 68.0 mm to (288.0, 508.0)
- moved C63 68.0 mm to (288.0, 516.0)
Connections:
- D10 pad 1: GND -> ISO_IN1_PTCA
- D10 pad 2: GOOBAY_CC1 -> ISO_GND1
- D11 pad 2: GOOBAY_CC2 -> GOOBAY_CC1
- D6 pad 1: USB_VBUS_1 -> USB_VBUS_1_FUSED
- D7 pad 1: USB_VBUS_4 -> USB_VBUS_4_FUSED
- D8 pad 1: USB_VBUS_5 -> USB_VBUS_5_FUSED
- D9 pad 1: ISO_IN1_PTCA -> RLY_COIL_N
- D9 pad 2: ISO_GND1 -> 3V3_SYS
- J1 pad 1: BAT -> BAT_PROTECTED
- J10 pad 2: HUB2_DN_DM_1 -> HUB2_DN_DM_1_SW
- J10 pad 3: HUB2_DN_DP_1 -> HUB2_DN_DP_1_SW
- J11 pad A6: HUB2_DN_DP_3 -> HUB2_DN_DP_3_SW
- J11 pad A7: HUB2_DN_DM_3 -> HUB2_DN_DM_3_SW
- J12 pad 3: ISO_IN1_RAW -> WAGO_COM1
- J12 pad 4: ISO_IN2_RAW -> WAGO_COM2
- J13 pad A4: IP5328P_VBUS -> GOOBAY_VBUS_FUSED
- J15 pad R1: SPK_N -> SPK_N_FUSED
- J15 pad T: SPK_P -> SPK_P_FUSED
- J17 pad 1: ADC_AIN0 -> ADC_AIN0_P
- J17 pad 2: ADC_AIN1 -> ADC_AIN1_P
- J17 pad 3: ADC_AIN2 -> ADC_AIN2_P
- J17 pad 4: ADC_AIN3 -> ADC_AIN3_P
- J3 pad 28: GND -> ISO_DO1
- J3 pad 34: GND -> WAGO_MODE
- J4 pad 1: ISO_DO1 -> 3V3_J4_OUT
- J4 pad 2: ISO_DO2 -> 5V_J4_OUT
- J4 pad 3: IR_GPIO -> AUX_GPIO_1_P
- J4 pad 4: AUX_GPIO_1 -> AUX_GPIO_2_P
- J4 pad 5: AUX_GPIO_2 -> AUX_GPIO_3_P
- J4 pad 6: AUX_GPIO_3 -> IR_GPIO_P
- J4 pad 7: GND -> RS485_A
- J4 pad 8: GND -> RS485_B
- J7 pad A6: HUB1_DN_DP_1 -> HUB1_DN_DP_1_SW
- J7 pad A7: HUB1_DN_DM_1 -> HUB1_DN_DM_1_SW
- J8 pad 2: HUB1_DN_DM_2 -> HUB1_DN_DM_2_SW
- J8 pad 3: HUB1_DN_DP_2 -> HUB1_DN_DP_2_SW
- J9 pad 2: HUB1_DN_DM_3 -> HUB1_DN_DM_3_SW
- J9 pad 3: HUB1_DN_DP_3 -> HUB1_DN_DP_3_SW
- Q4 pad 1: IR_GPIO -> WAGO_MODE
- Q4 pad 2: IR_LED_N -> GND
- Q4 pad 3: GND -> RLY_COIL_N
- R34 pad 1: ISO_IN1_PTCA -> WAGO_MODE
- R34 pad 2: ISO_IN1 -> GND
- R35 pad 1: ISO_SENSE1 -> ISO_IN1_PTCA
- R35 pad 2: ISO_GND1 -> ISO_IN1
- R36 pad 1: ISO_IN2_PTCA -> ISO_SENSE1
- R36 pad 2: ISO_IN2 -> ISO_GND1
- R37 pad 1: ISO_SENSE2 -> ISO_IN2_PTCA
- R37 pad 2: ISO_GND1 -> ISO_IN2
- R38 pad 1: RTL_RSET -> ISO_SENSE2
- R38 pad 2: GND -> ISO_GND1
- R39 pad 1: 3V3_CLEAN -> RTL_RSET
- R39 pad 2: RTL_LANWAKEB -> GND
- R40 pad 1: 3V3_SYS -> 3V3_CLEAN
- R40 pad 2: SPI3_CS -> RTL_LANWAKEB
- R41 pad 2: NAV_UP -> SPI3_CS
- R42 pad 2: NAV_DOWN -> NAV_UP
- R43 pad 2: NAV_LEFT -> NAV_DOWN
- R44 pad 2: NAV_RIGHT -> NAV_LEFT
- R45 pad 2: NAV_CENTER -> NAV_RIGHT
- R46 pad 2: PCF8574_INT -> NAV_CENTER
- R47 pad 1: 5V_SYS -> 3V3_SYS
- R47 pad 2: IR_LED_P -> PCF8574_INT
- R48 pad 1: IR_GPIO -> 5V_SYS
- R48 pad 2: GND -> IR_LED_P
- R49 pad 1: I2S_DATA_IN -> IR_GPIO
- R50 pad 1: 3V3_SYS -> I2S_DATA_IN
- R50 pad 2: AMP_SD -> GND
- R51 pad 1: AMP_OUT_P -> 3V3_SYS
- R51 pad 2: AMP_OUT_P_FILT -> AMP_SD
- R52 pad 1: AMP_OUT_N -> AMP_OUT_P
- R52 pad 2: AMP_OUT_N_FILT -> AMP_OUT_P_FILT
- R53 pad 1: TRRS_DETECT_RAW -> AMP_OUT_N
- R53 pad 2: AMP_SD -> AMP_OUT_N_FILT
- R54 pad 1: MIC_VDD -> TRRS_DETECT_RAW
- R54 pad 2: MIC_LED_A -> AMP_SD
- R55 pad 1: 3V3_SYS -> MIC_VDD
- R55 pad 2: PWR_LED_A -> MIC_LED_A
- R56 pad 2: PMIC_LIGHT_LED -> PWR_LED_A
- R57 pad 1: CODEC_LMICN -> 3V3_SYS
- R57 pad 2: GND -> PMIC_LIGHT_LED
- R58 pad 1: CODEC_ADCOUT -> CODEC_LMICN
- R58 pad 2: I2S_DATA_IN -> GND
- R59 pad 1: CODEC_MICBIAS -> CODEC_ADCOUT
- R59 pad 2: TRRS_RING2 -> I2S_DATA_IN
- R60 pad 1: ADC_ADDR -> CODEC_MICBIAS
- R60 pad 2: GND -> TRRS_RING2
- R61 pad 1: 3V3_SYS -> ADC_ADDR
- R61 pad 2: ADC_ALRT -> GND
- R62 pad 1: AUX_GPIO_3 -> 3V3_SYS
- R62 pad 2: RS485_DE -> ADC_ALRT
- R63 pad 1: RS485_DE -> AUX_GPIO_3
- R63 pad 2: GND -> RS485_DE
- R64 pad 1: RS485_A -> RS485_DE
- R64 pad 2: RS485_B -> GND
- R65 pad 1: 3V3_SYS -> RS485_A
- R65 pad 2: IR_VS_FILT -> RS485_B
- U12 pad 1: HUB1_DN_DM_1 -> HUB1_DN_DM_1_SW
- U12 pad 3: HUB1_DN_DM_1 -> HUB1_DN_DM_1_SW
- U12 pad 4: HUB1_DN_DP_1 -> HUB1_DN_DP_1_SW
- U12 pad 6: HUB1_DN_DP_1 -> HUB1_DN_DP_1_SW
- U16 pad 1: HUB1_DN_DM_2 -> HUB1_DN_DM_2_SW
- U16 pad 3: HUB1_DN_DM_2 -> HUB1_DN_DM_2_SW
- U16 pad 4: HUB1_DN_DP_2 -> HUB1_DN_DP_2_SW
- U16 pad 6: HUB1_DN_DP_2 -> HUB1_DN_DP_2_SW
- U17 pad 1: HUB1_DN_DM_3 -> HUB1_DN_DM_3_SW
- U17 pad 3: HUB1_DN_DM_3 -> HUB1_DN_DM_3_SW
- U17 pad 4: HUB1_DN_DP_3 -> HUB1_DN_DP_3_SW
- U17 pad 6: HUB1_DN_DP_3 -> HUB1_DN_DP_3_SW
- U18 pad 1: HUB2_DN_DM_1 -> HUB2_DN_DM_1_SW
- U18 pad 3: HUB2_DN_DM_1 -> HUB2_DN_DM_1_SW
- U18 pad 4: HUB2_DN_DP_1 -> HUB2_DN_DP_1_SW
- U18 pad 6: HUB2_DN_DP_1 -> HUB2_DN_DP_1_SW
- U19 pad 1: HUB2_DN_DM_3 -> HUB2_DN_DM_3_SW
- U19 pad 3: HUB2_DN_DM_3 -> HUB2_DN_DM_3_SW
- U19 pad 4: HUB2_DN_DP_3 -> HUB2_DN_DP_3_SW
- U19 pad 6: HUB2_DN_DP_3 -> HUB2_DN_DP_3_SW
