File: daemon_v0.kicad_pcb (KiCad board)
At the start: 4 copper layers, 86 x 53 mm, 338 parts, among them J1 Battery PTC 2A Fuse, J10 USB-A♂ Charge Port 4, J11 USB-C♀ Main Port 5, J12 WAGO 4P Field Terminal, J13 USB-C♀ Goobay Bridge, J14 RJ45 MagJack, J15 TRRS 3.5mm Jack, J16 Speaker JST, J17 Analog-In, J2 10mΩ Current Sense, J3 40-Pin Radxa Header, J4 AUX GPIO Breakout, J6 ST7789 SPI Display, J7 USB-C♂ Plug → Radxa (KEY), J8 USB-A♀ Host Port 2, J9 USB-A♀ Host Port 3, K1 G6K-2F-Y, Q1 BC857 Dummy Load PNP, Q2 BSS84 Wake PMOS, Q3 2N7002 PMIC Kill NMOS, Q4 AO3400A IR Drive NMOS, Q5 AO3400A, SW1 Power Button, SW2 5-Way Nav Switch, U1 IP5328P PMIC, U10 MAX98357A I2S Amp, U11 ISO1212 Dual Isolator, U12 ESD USB Port1, U13 INMP441 Mic Left, U14 SL2.1A USB Hub 2, U15 SY6280 Port4 USB-A♂, U16 ESD USB Port2, U17 ESD USB Port3, U18 ESD USB Port4, U19 ESD USB Port5, U2 AP2112K 3.3V LDO, U20 ESD Goobay Bridge, U21 PCF8574 I2C GPIO Exp, U22 SY6280 Port5 USB-C♀, U23 3.3→5V Level Shifter, U24 INMP441 Mic Right, U25 ESD9B5.0ST5G, U26 ESD9B5.0ST5G, U27 NAU88C22, U28 ADS1115, U29 SP3485, U3 SL2.1A USB Hub 1, U30 TSOP38238, U31 ATECC608B, U32 74LVC04A, U33 TS3USB221, U34 TS3USB221, U35 TS3USB221, U36 TS3USB221, U37 TS3USB221, U4 SY6280 Port1 Radxa Key, U5 SY6280 Port2 USB-A♀, U6 SY6280 Port3 USB-A♀, U7 NE555 Heartbeat Timer, U8 CC1101 Sub-GHz Radio, U9 RTL8152B Ethernet, Y1 12MHz Hub1 Xtal, Y2 12MHz Hub2 Xtal, Y3 27MHz CC1101 Xtal, Y4 25MHz Ethernet Xtal

Commit message: fix: flip J6 screen connector to B.Cu — female socket on back side
Parts:
- J6: moved to B.Cu
- turned J6 to -90 degrees

Commit message: fix: J6 screen connector — PinHeader through-hole pads for Mill-Max receptacles
Parts:
- J6: footprint PinSocket_1x08_P2.54mm_Vertical -> PinHeader_1x08_P2.54mm_Vertical; moved to F.Cu
- turned J6 to 90 degrees
